Commit message: feat: validate Gazebo SLAM and add Nav2 end-to-end harness

File: ros2_ws/src/homeagent_description/urdf/homebot.urdf.xacro (robot description, xacro)
@@ -1,4 +1,5 @@
 <?xml version="1.0"?>
 <robot xmlns:xacro="http://www.ros.org/wiki/xacro" name="homebot">
+  <link name="base_footprint"/>
   <link name="base_link">
     <inertial>
@@ -13,4 +14,9 @@
     <collision><geometry><box size="0.42 0.32 0.14"/></geometry></collision>
   </link>
+  <joint name="base_footprint_joint" type="fixed">
+    <parent link="base_footprint"/>
+    <child link="base_link"/>
+    <origin xyz="0 0 0" rpy="0 0 0"/>
+  </joint>
   <link name="left_wheel_link">
     <inertial>
@@ -86,5 +92,5 @@
     <parent link="base_link"/>
     <child link="lidar_link"/>
-    <origin xyz="0.02 0 0.11"/>
+    <origin xyz="0.02 0 0.30"/>
   </joint>
   <link name="camera_link">
@@ -121,5 +127,5 @@
       <odometry_topic>odom</odometry_topic>
       <odometry_frame>odom</odometry_frame>
-      <robot_base_frame>base_link</robot_base_frame>
+      <robot_base_frame>base_footprint</robot_base_frame>
       <publish_odom>true</publish_odom>
       <publish_odom_tf>true</publish_odom_tf>
