Commit message: feat: add gripper control and logical pick attachment

File: ros2_ws/src/homeagent_manipulation/config/homearm.urdf.xacro (robot description, xacro)
@@ -139,4 +139,38 @@
     <origin xyz="0.16 0 0"/>
   </joint>
+  <link name="gripper_fixed_finger_link">
+    <visual>
+      <origin xyz="0.05 0 0"/>
+      <geometry><box size="0.10 0.012 0.03"/></geometry>
+      <material name="gray"/>
+    </visual>
+    <collision>
+      <origin xyz="0.05 0 0"/>
+      <geometry><box size="0.10 0.012 0.03"/></geometry>
+    </collision>
+  </link>
+  <joint name="gripper_fixed_finger_joint" type="fixed">
+    <parent link="tool_link"/>
+    <child link="gripper_fixed_finger_link"/>
+    <origin xyz="0.07 -0.025 0"/>
+  </joint>
+  <link name="gripper_finger_link">
+    <visual>
+      <origin xyz="0.05 0 0"/>
+      <geometry><box size="0.10 0.012 0.03"/></geometry>
+      <material name="gray"/>
+    </visual>
+    <collision>
+      <origin xyz="0.05 0 0"/>
+      <geometry><box size="0.10 0.012 0.03"/></geometry>
+    </collision>
+  </link>
+  <joint name="gripper_joint" type="prismatic">
+    <parent link="tool_link"/>
+    <child link="gripper_finger_link"/>
+    <origin xyz="0.07 0.025 0"/>
+    <axis xyz="0 1 0"/>
+    <limit lower="0.0" upper="0.04" effort="20" velocity="0.08"/>
+  </joint>
   <ros2_control name="HomeArmSystem" type="system">
     <hardware>
@@ -172,4 +206,11 @@
       <state_interface name="velocity"/>
     </joint>
+    <joint name="gripper_joint">
+      <command_interface name="position"/>
+      <state_interface name="position">
+        <param name="initial_value">0.04</param>
+      </state_interface>
+      <state_interface name="velocity"/>
+    </joint>
   </ros2_control>
 </robot>

Commit message: feat: integrate Nav2 and MoveIt mobile manipulator demo

File: ros2_ws/src/homeagent_manipulation/config/homearm.urdf.xacro (robot description, xacro)
@@ -4,6 +4,6 @@
   <material name="blue"><color rgba="0.12 0.35 0.75 1"/></material>
   <material name="orange"><color rgba="0.9 0.45 0.08 1"/></material>
-  <link name="base_footprint"/>
-  <link name="base_link">
+  <link name="arm_base_footprint"/>
+  <link name="arm_base_link">
     <visual>
       <origin xyz="0 0 0.04"/>
@@ -21,7 +21,7 @@
     </inertial>
   </link>
-  <joint name="base_footprint_joint" type="fixed">
-    <parent link="base_footprint"/>
-    <child link="base_link"/>
+  <joint name="arm_base_footprint_joint" type="fixed">
+    <parent link="arm_base_footprint"/>
+    <child link="arm_base_link"/>
     <origin xyz="0 0 0" rpy="0 0 0"/>
   </joint>
@@ -43,5 +43,5 @@
   </link>
   <joint name="joint1" type="revolute">
-    <parent link="base_link"/>
+    <parent link="arm_base_link"/>
     <child link="shoulder_link"/>
     <origin xyz="0 0 0.08" rpy="0 0 0"/>
